File: HappySwitchV2/HappySwitchV2.kicad_pcb (KiCad board)
At the start: 2 copper layers, 210.1 x 55.3 mm, 42 parts, among them J1 DIN-8, J2 DIN-5_180degree, Q1 4N25-X007T, SW1 SW_Push, SW2 SW_Push, SW3 SW_Push, SW4 SW_Push, SW5 SW_Push, U1 Sparkfun_Pro_Micro

Commit message: Add files via upload
Parts:
- PWR: renamed from GND; value 5V+ -> USB PWR
- R17, R18: value 220 -> R220
- R4: value R 220 -> R220
- R8: value 470 -> R470
Connections:
- PWR pad 1: GND -> Arduino_D15
- PWR pad 2: +5V -> GND
Routing:
- net GND: track 0.00 -> 174.0 mm, vias 63 -> 65
- net +5V: track 174.0 -> 0.00 mm, vias 2 -> 0
