File: HappySwitchV2/HappySwitchV2.kicad_sch (KiCad schematic)
At the start: 41 parts, among them J1 DIN-8, J2 DIN-5_180degree, Q1 4N25-X007T, SW1 SW_Push, SW2 SW_Push, SW3 SW_Push, SW4 SW_Push, SW5 SW_Push, U1 Sparkfun_Pro_Micro

Commit message: Add files via upload
Parts:
- D1, D5, D6: DigiKey Part Number  (none) -> 4878-1N4148WCT-ND; MPN (none) -> 1N4148W; Manufacturer (none) -> Diotec Semiconductor
- Q1: DigiKey Part Number  (none) -> 4N25-X007TCT-ND; MPN (none) -> 4N25-X007T; Manufacturer (none) -> Vishay Semiconductor Opto Division
- R1, R10, R15, R16, R19, R2, R20, R21, R22, R23, R3: DigiKey Part Number  (none) -> 10-ERA-6VEB1002VCT-ND; MPN (none) -> ERA-6VEB1002V; Manufacturer (none) -> Panasonic Electronic Components
- R11, R14: DigiKey Part Number  (none) -> P21076CT-ND; MPN (none) -> ERJ-PB6D3301V; Manufacturer (none) -> Panasonic Electronic Components
- R12: DigiKey Part Number  (none) -> P20676CT-ND; MPN (none) -> ERJ-PB6B5231V; Manufacturer (none) -> Panasonic Electronic Components
- R13: DigiKey Part Number  (none) -> 10-ERA-6VEB1003VCT-ND; MPN (none) -> ERA-6VEB1003V; Manufacturer (none) -> Panasonic Electronic Components
- R17, R18: value 220 -> R220; DigiKey Part Number  (none) -> P20516CT-ND; MPN (none) -> ERJ-PB6B2200V; Manufacturer (none) -> Panasonic Electronic Components
- R25: DigiKey Part Number  (none) -> P0.0ACT-ND; MPN (none) -> ERJ-6GEY0R00V; Manufacturer (none) -> Panasonic Electronic Components
- R4: value R 220 -> R220; DigiKey Part Number  (none) -> P20516CT-ND; MPN (none) -> ERJ-PB6B2200V; Manufacturer (none) -> Panasonic Electronic Components
- R5, R6, R7: DigiKey Part Number  (none) -> P20516CT-ND; MPN (none) -> ERJ-PB6B2200V; Manufacturer (none) -> Panasonic Electronic Components
- R8: value 470 -> R470; DigiKey Part Number  (none) -> 10-ERA-6VEB4700VCT-ND; MPN (none) -> ERA-6VEB4700V; Manufacturer (none) -> Panasonic Electronic Components
- R9: DigiKey Part Number  (none) -> 10-ERA-6VEB4701VCT-ND; MPN (none) -> ERA-6VEB4701V; Manufacturer (none) -> Panasonic Electronic Components
